File: linklet.kicad_pcb (KiCad board)
At the start: 4 copper layers, 61 x 36 mm, 42 parts, among them J1 USB_B_Micro, J2 Conn_01x04_Pin, J3 Conn_01x04_Pin, J4 Conn_01x04_Pin, J6 Conn_Coaxial, J7 Conn_01x08_Socket, SW1 SW_SPDT, U1 STM32F103C8T6, U2 AMS1117-3.3, U3 RFM69HCW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

Commit message: update silkscreen
Parts:
- added G***: LOGO, LOGO, F.Cu at (109.0, 89.0)
- moved R8 0.90 mm to (91.2, 85.5)
- moved R9 0.90 mm to (93.8, 85.5)
Routing:
- net /USER_I2C_SCL: track 19.0 -> 19.9 mm
- net /USER_I2C_SDA: track 13.6 -> 14.5 mm
Other:
- board text added: "GND NC NC TX RX SCL SDA VCC"
- board text added: "I2C"
- board text added: "PWR"
- board text added: "Rx"
- board text added: "SWD"
- board text added: "Tx"
- board text added: "UART"
- board text added: "← = 1"
