File: linklet.kicad_pcb (KiCad board)
At the start: 4 copper layers, 61 x 36 mm, 43 parts, among them J1 USB_B_Micro, J2 Conn_01x04_Pin, J3 Conn_01x04_Pin, J4 Conn_01x04_Pin, J6 Conn_Coaxial, J7 Conn_01x08_Socket, SW1 SW_SPDT, U1 STM32F103C8T6, U2 AMS1117-3.3, U3 RFM69HCW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

Commit message: add manufacturing files
Parts:
- added FID1: Fiducial, Fiducial:Fiducial_1mm_Mask2mm, F.Cu at (109.8, 112.5)
- added FID2: Fiducial, Fiducial:Fiducial_1mm_Mask2mm, F.Cu at (99.0, 86.6)
- added FID3: Fiducial, Fiducial:Fiducial_1mm_Mask2mm, F.Cu at (76.6, 98.8)
- D2: value BLUE -> RED
- D3: value GREEN -> RED
- FB1: value 120R -> 220R
Connections:
- net Net-(J6-In) renamed /RFM69HCW_ANT
Routing:
- net /USER_I2C_SCL: track 19.9 -> 19.0 mm
- net /USER_I2C_SDA: track 14.5 -> 13.6 mm
- net GND: vias 30 -> 33
- net (no net): vias 3 -> 0
- added copper zone on F.Cu, net /RFM69HCW_ANT
