File: linklet.kicad_sch (KiCad schematic)
At the start: 42 parts, among them J1 USB_B_Micro, J2 Conn_01x04_Pin, J3 Conn_01x04_Pin, J4 Conn_01x04_Pin, J6 Conn_Coaxial, J7 Conn_01x08_Socket, SW1 SW_SPDT, U1 STM32F103C8T6, U2 AMS1117-3.3, U3 RFM69HCW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

Commit message: add manufacturing files
Parts:
- added FID1, FID2, FID3: Fiducial, Fiducial:Fiducial_1mm_Mask2mm, symbol Mechanical:Fiducial
- C1, C2, C3, C4, C9: LCSC PN (none) -> C309458
- C10, C11: LCSC PN (none) -> C106199
- C12, C13: LCSC PN (none) -> C452754
- C5: LCSC PN (none) -> C96446
- C6: LCSC PN (none) -> C3855387
- C7, C8: LCSC PN (none) -> C52923
- D1: LCSC PN (none) -> C965798
- D2: value BLUE -> RED; LCSC PN (none) -> C965798
- D3: value GREEN -> RED; LCSC PN (none) -> C965798
- FB1: value 120R -> 220R; LCSC PN (none) -> C66810
- J1: LCSC PN (none) -> C2894326
- J2, J3, J4: LCSC PN (none) -> C5116483
- J6: LCSC PN (none) -> C43302011
- J7: LCSC PN (none) -> C9900212703
- R1: LCSC PN (none) -> C1002
- R2, R3, R4, R5, R8, R9: LCSC PN (none) -> C25867
- R6, R7: LCSC PN (none) -> C49652832
- SW1: LCSC PN (none) -> C221841
- U1: LCSC PN (none) -> C8734
- U2: LCSC PN (none) -> C6186
- U3: now not fitted
- Y1: LCSC PN (none) -> C112972
Connections:
- net RFM69HCW_ANT: now reaches J6.1 (In), U3.9 (ANT)
Other:
- note added: "Fiducials"
- moved on the sheet: J6
